File: kicad/servo_controller/servo_controller.kicad_pcb (KiCad board)
At the start: 2 copper layers, 24 parts, among them J1 Conn_01x03_Male, J2 Conn_01x02_Male, SW1 Rotary_Encoder_Switch, U1 LM2576HVT-5, U2 HDSP-A153, U3 74HCT541, U4 ProMicro, U5 NCP1117-5.0_SOT223

Commit message: Migrating to KiCad6
Other:
- net class Default removed
