File: kicad/tda2030a/tda2030a.kicad_pcb (KiCad board)
At the start: 2 copper layers, 32 x 24 mm, 19 parts, among them J1 Conn_01x04_Male, J2 Conn_01x02_Female, U1 TDA2030

Commit message: Migrating to KiCad6
Other:
- net class Default removed
