File: kicad/mic_amp/mic_amp.kicad_pcb (KiCad board)
At the start: 2 copper layers, 136 x 80 mm, 70 parts, among them J1 AudioJack3_Dual_Switch, J2 AudioJack3_Dual_Switch, J3 Conn_01x02_Male, J4 Conn_01x02_Male, J5 Conn_01x04_Female, P101 R_POT_Dual, P201 R_POT_Dual, SW1 SW_DPDT_x2, U1 NE5532DR, U101 NE5532DR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

Commit message: Migrating to KiCad6
Connections:
- J1 pad R1: Net-(J1-PadR1) -> unconnected-(J1-PadR1)
- J1 pad R2: Net-(J1-PadR2) -> unconnected-(J1-PadR2)
- J1 pad RN1: Net-(J1-PadRN1) -> unconnected-(J1-PadRN1)
- J1 pad RN2: Net-(J1-PadRN2) -> unconnected-(J1-PadRN2)
- J1 pad SN1: Net-(J1-PadSN1) -> unconnected-(J1-PadSN1)
- J1 pad SN2: Net-(J1-PadSN2) -> unconnected-(J1-PadSN2)
- J1 pad TN1: Net-(J1-PadTN1) -> unconnected-(J1-PadTN1)
- J1 pad TN2: Net-(J1-PadTN2) -> unconnected-(J1-PadTN2)
- J2 pad RN1: Net-(J2-PadRN1) -> unconnected-(J2-PadRN1)
- J2 pad RN2: Net-(J2-PadRN2) -> unconnected-(J2-PadRN2)
- J2 pad SN1: Net-(J2-PadSN1) -> unconnected-(J2-PadSN1)
- J2 pad SN2: Net-(J2-PadSN2) -> unconnected-(J2-PadSN2)
- J2 pad TN1: Net-(J2-PadTN1) -> unconnected-(J2-PadTN1)
- J2 pad TN2: Net-(J2-PadTN2) -> unconnected-(J2-PadTN2)
- SW1 pad 6: Net-(SW1-Pad6) -> unconnected-(SW1-Pad6)
Other:
- net class Default removed
