File: kicad/mic_amp/mic_amp.kicad_sch (KiCad schematic)
At the start: 70 parts

Commit message: Migrating to KiCad 9
Parts:
- C1, C10, C3: value (none) -> 1uF; footprint (none) -> Capacitor_SMD:C_0805_2012Metric
- C101, C102, C106, C201, C202, C206: value (none) -> 4.7uF, 16V; footprint (none) -> Capacitor_SMD:CP_Elec_4x5.4
- C103, C107, C203, C207: value (none) -> 22pF; footprint (none) -> Capacitor_SMD:C_0805_2012Metric
- C104, C105, C108, C204, C205, C208: value (none) -> 220uF, 16V; footprint (none) -> Capacitor_SMD:CP_Elec_6.3x7.7
- C11: value (none) -> 10uF, 16V; footprint (none) -> Capacitor_SMD:CP_Elec_4x5.4
- C2, C4: value (none) -> 1nF; footprint (none) -> Capacitor_SMD:C_0805_2012Metric
- C5, C6: value (none) -> 0.1nF; footprint (none) -> Capacitor_SMD:C_0805_2012Metric
- C7, C9: value (none) -> 22uF, 16V; footprint (none) -> Capacitor_SMD:CP_Elec_5x5.4
- C8: value (none) -> 6.8nF; footprint (none) -> Capacitor_SMD:C_0805_2012Metric
- D1, D2: value (none) -> LED; footprint (none) -> LED_THT:LED_D3.0mm_Horizontal_O3.81mm_Z6.0mm
- J1, J2: value (none) -> AudioJack3_Dual_Switch; footprint (none) -> lib:CK635-037
- J3: value (none) -> Conn_01x02_Male; footprint (none) -> Connector_JST:JST_PH_B2B-PH-K_1x02_P2.00mm_Vertical
- J4: value (none) -> Conn_01x02_Male; footprint (none) -> Connector_JST:JST_XH_B2B-XH-A_1x02_P2.50mm_Vertical
- J5: value (none) -> Conn_01x04_Female; footprint (none) -> Connector_PinSocket_2.54mm:PinSocket_1x04_P2.54mm_Vertical
- L1: value (none) -> 1mH; footprint (none) -> Inductor_THT:L_Radial_D7.8mm_P5.00mm_Fastron_07HCP
- P101, P201: value (none) -> R_POT_Dual; footprint (none) -> Potentiometer_THT:Potentiometer_Alps_RK097_Dual_Horizontal
- R1: value (none) -> 1k; footprint (none) -> Potentiometer_THT:Potentiometer_Bourns_3339P_Vertical
- R10, R11, R9: value (none) -> 1k; footprint (none) -> Resistor_SMD:R_0805_2012Metric
- R101, R105, R201, R205: value (none) -> 18k; footprint (none) -> Resistor_SMD:R_1206_3216Metric
- R102, R103, R104, R106, R202, R203, R204, R206: value (none) -> 68k; footprint (none) -> Resistor_SMD:R_1206_3216Metric
- R12, R13, R5, R6, R7, R8: value (none) -> 10k; footprint (none) -> Resistor_SMD:R_0805_2012Metric
- R14: value (none) -> 2k; footprint (none) -> Resistor_SMD:R_0805_2012Metric
- R15: value (none) -> R_POT; footprint (none) -> Connector_JST:JST_PH_B3B-PH-K_1x03_P2.00mm_Vertical
- R16: value (none) -> 100k; footprint (none) -> Resistor_SMD:R_0805_2012Metric
- R17: value (none) -> 15k; footprint (none) -> Resistor_SMD:R_0805_2012Metric
- R2, R3: value (none) -> 4.7k; footprint (none) -> Resistor_SMD:R_0805_2012Metric
- R4: value (none) -> 39; footprint (none) -> Resistor_SMD:R_0805_2012Metric
- SW1: value (none) -> SW_DPDT_x2; footprint (none) -> lib:MTS-202-C3_DPDT_Angled
- U1, U101, U201: value (none) -> NE5532DR; footprint (none) -> Package_SO:SOIC-8_3.9x4.9mm_P1.27mm
